Commit message: First commit

File: panda_gripper.urdf (robot description, URDF)
Before this commit: robot gripper, 2 links, 1 joints
Links:
- removed link finger1
- removed link finger2
- added link panda_hand; collision mesh filename=franka_description/meshes/collision/hand.stl; visual mesh filename=franka_description/meshes/visual/hand.dae
- added link panda_leftfinger; collision mesh filename=franka_description/meshes/collision/finger.stl; visual mesh filename=franka_description/meshes/visual/finger.dae
- added link panda_rightfinger; collision mesh filename=franka_description/meshes/collision/finger.stl; visual mesh filename=franka_description/meshes/visual/finger.dae
Joints:
- removed joint finger1_joint
- added joint panda_finger_joint1: type prismatic, parent panda_hand, child panda_leftfinger, origin xyz=0 0 0.0584 rpy=0 0 0, axis 0 1 0, limit lower=0.0 upper=0.04 effort=20 velocity=0.2
- added joint panda_finger_joint2: type prismatic, parent panda_hand, child panda_rightfinger, origin xyz=0 0 0.0584 rpy=0 0 0, axis 0 -1 0, limit lower=0.0 upper=0.04 effort=20 velocity=0.2, mimic joint=panda_finger_joint1
